Commit message: Refactor RL agent evaluation and training scripts for Isaac Lab compatibility
- Updated `eval_agent_trl.py` to integrate argparse for command-line arguments and removed legacy version checks for IsaacSim.
- Enhanced startup hold functionality in `base_sim.py` to stabilize robot initialization and added new configuration parameters for startup behavior.
- Modified `train_agent_trl.py` to align with new visualizer selection methods in Isaac Lab 3.x.
- Introduced new command-line arguments in `run_isaacsim_loop.py` to control startup hold behavior.
- Updated dependencies in `pyproject.toml` to support NumPy 2 for Python 3.12.
- Added elastic band wrench calculations in `control.py` for improved root suspension during startup.
- Implemented unit tests for new startup hold features and elastic band wrench functionality in `test_contract.py`.
- Created a backup robot configuration file for G1 robot with detailed actuator settings and mappings.

File: gear_sonic/data/assets/robot_description/urdf/g1/main.urdf (robot description, URDF)
Before this commit: robot g1, 54 links, 53 joints
Links:
- link head_link: geometry visual mesh filename=/home/tuan/projects/cibo/3rd_party/GR00T-WholeBodyControl/g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
- link left_ankle_pitch_link: geometry visual mesh filename=/home/tuan/projects/cibo/3rd_party/GR00T-WholeBodyControl/g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
- link left_ankle_roll_link: geometry collision cylinder length=0.05 radius=0.01; collision cylinder length=0.05 radius=0.01
- link left_elbow_link: geometry collision cylinder length=0.13 radius=0.035; visual mesh filename=/home/tuan/projects/cibo/3rd_party/GR00T-WholeBodyControl/g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
- link left_hand_index_0_link: geometry collision mesh filename=/home/tuan/projects/cibo/3rd_party/GR00T-WholeBodyControl/g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; visual mesh filename=/home/tuan/projects/cibo/3rd_party/GR00T-WholeBodyControl/g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
- link left_hand_index_1_link: geometry collision mesh filename=/home/tuan/projects/cibo/3rd_party/GR00T-WholeBodyControl/g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; visual mesh filename=/home/tuan/projects/cibo/3rd_party/GR00T-WholeBodyControl/g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
- link left_hand_middle_0_link: geometry collision mesh filename=/home/tuan/projects/cibo/3rd_party/GR00T-WholeBodyControl/g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; visual mesh filename=/home/tuan/projects/cibo/3rd_party/GR00T-WholeBodyControl/g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
- link left_hand_middle_1_link: geometry collision mesh filename=/home/tuan/projects/cibo/3rd_party/GR00T-WholeBodyControl/g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; visual mesh filename=/home/tuan/projects/cibo/3rd_party/GR00T-WholeBodyControl/g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
- link left_hand_palm_link: geometry collision mesh filename=/home/tuan/projects/cibo/3rd_party/GR00T-WholeBodyControl/g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; visual mesh filename=/home/tuan/projects/cibo/3rd_party/GR00T-WholeBodyControl/g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
- link left_hand_thumb_0_link: geometry collision mesh filename=/home/tuan/projects/cibo/3rd_party/GR00T-WholeBodyControl/g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; visual mesh filename=/home/tuan/projects/cibo/3rd_party/GR00T-WholeBodyControl/g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
- link left_hand_thumb_1_link: geometry collision mesh filename=/home/tuan/projects/cibo/3rd_party/GR00T-WholeBodyControl/g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; visual mesh filename=/home/tuan/projects/cibo/3rd_party/GR00T-WholeBodyControl/g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
- link left_hand_thumb_2_link: geometry collision mesh filename=/home/tuan/projects/cibo/3rd_party/GR00T-WholeBodyControl/g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; visual mesh filename=/home/tuan/projects/cibo/3rd_party/GR00T-WholeBodyControl/g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
- link left_hip_pitch_link: geometry visual mesh filename=/home/tuan/projects/cibo/3rd_party/GR00T-WholeBodyControl/g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
- link left_hip_roll_link: geometry collision cylinder length=0.2 radius=0.05; visual mesh filename=/home/tuan/projects/cibo/3rd_party/GR00T-WholeBodyControl/g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
- link left_hip_yaw_link: geometry visual mesh filename=/home/tuan/projects/cibo/3rd_party/GR00T-WholeBodyControl/g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
- link left_knee_link: geometry collision cylinder length=0.2 radius=0.05; visual mesh filename=/home/tuan/projects/cibo/3rd_party/GR00T-WholeBodyControl/g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
- link left_shoulder_pitch_link: geometry visual mesh filename=/home/tuan/projects/cibo/3rd_party/GR00T-WholeBodyControl/g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
- link left_shoulder_roll_link: geometry visual mesh filename=/home/tuan/projects/cibo/3rd_party/GR00T-WholeBodyControl/g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
- link left_shoulder_yaw_link: geometry collision cylinder length=0.13 radius=0.035; visual mesh filename=/home/tuan/projects/cibo/3rd_party/GR00T-WholeBodyControl/g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
- link left_wrist_pitch_link: geometry visual mesh filename=/home/tuan/projects/cibo/3rd_party/GR00T-WholeBodyControl/g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
- link left_wrist_roll_link: geometry visual mesh filename=/home/tuan/projects/cibo/3rd_party/GR00T-WholeBodyControl/g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
- link left_wrist_yaw_link: geometry collision mesh filename=/home/tuan/projects/cibo/3rd_party/GR00T-WholeBodyControl/g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; visual mesh filename=/home/tuan/projects/cibo/3rd_party/GR00T-WholeBodyControl/g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
- link logo_link: geometry visual mesh filename=/home/tuan/projects/cibo/3rd_party/GR00T-WholeBodyControl/g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
- link pelvis: geometry collision sphere radius=0.07; visual mesh filename=/home/tuan/projects/cibo/3rd_party/GR00T-WholeBodyControl/g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
- link pelvis_contour_link: geometry visual mesh filename=/home/tuan/projects/cibo/3rd_party/GR00T-WholeBodyControl/g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
- link right_ankle_pitch_link: geometry visual mesh filename=/home/tuan/projects/cibo/3rd_party/GR00T-WholeBodyControl/g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
- link right_ankle_roll_link: geometry collision cylinder length=0.05 radius=0.01; collision cylinder length=0.05 radius=0.01
- link right_elbow_link: geometry collision cylinder length=0.13 radius=0.035; visual mesh filename=/home/tuan/projects/cibo/3rd_party/GR00T-WholeBodyControl/g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
- link right_hand_index_0_link: geometry collision mesh filename=/home/tuan/projects/cibo/3rd_party/GR00T-WholeBodyControl/g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; visual mesh filename=/home/tuan/projects/cibo/3rd_party/GR00T-WholeBodyControl/g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
- link right_hand_index_1_link: geometry collision mesh filename=/home/tuan/projects/cibo/3rd_party/GR00T-WholeBodyControl/g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; visual mesh filename=/home/tuan/projects/cibo/3rd_party/GR00T-WholeBodyControl/g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
- link right_hand_middle_0_link: geometry collision mesh filename=/home/tuan/projects/cibo/3rd_party/GR00T-WholeBodyControl/g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; visual mesh filename=/home/tuan/projects/cibo/3rd_party/GR00T-WholeBodyControl/g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
- link right_hand_middle_1_link: geometry collision mesh filename=/home/tuan/projects/cibo/3rd_party/GR00T-WholeBodyControl/g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; visual mesh filename=/home/tuan/projects/cibo/3rd_party/GR00T-WholeBodyControl/g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
- link right_hand_palm_link: geometry collision mesh filename=/home/tuan/projects/cibo/3rd_party/GR00T-WholeBodyControl/g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; visual mesh filename=/home/tuan/projects/cibo/3rd_party/GR00T-WholeBodyControl/g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
- link right_hand_thumb_0_link: geometry collision mesh filename=/home/tuan/projects/cibo/3rd_party/GR00T-WholeBodyControl/g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; visual mesh filename=/home/tuan/projects/cibo/3rd_party/GR00T-WholeBodyControl/g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
- link right_hand_thumb_1_link: geometry collision mesh filename=/home/tuan/projects/cibo/3rd_party/GR00T-WholeBodyControl/g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; visual mesh filename=/home/tuan/projects/cibo/3rd_party/GR00T-WholeBodyControl/g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
- link right_hand_thumb_2_link: geometry collision mesh filename=/home/tuan/projects/cibo/3rd_party/GR00T-WholeBodyControl/g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; visual mesh filename=/home/tuan/projects/cibo/3rd_party/GR00T-WholeBodyControl/g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
- link right_hip_pitch_link: geometry visual mesh filename=/home/tuan/projects/cibo/3rd_party/GR00T-WholeBodyControl/g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
- link right_hip_roll_link: geometry collision cylinder length=0.2 radius=0.05; visual mesh filename=/home/tuan/projects/cibo/3rd_party/GR00T-WholeBodyControl/g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
- link right_hip_yaw_link: geometry visual mesh filename=/home/tuan/projects/cibo/3rd_party/GR00T-WholeBodyControl/g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
- link right_knee_link: geometry collision cylinder length=0.2 radius=0.05; visual mesh filename=/home/tuan/projects/cibo/3rd_party/GR00T-WholeBodyControl/g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
- link right_shoulder_pitch_link: geometry visual mesh filename=/home/tuan/projects/cibo/3rd_party/GR00T-WholeBodyControl/g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
- link right_shoulder_roll_link: geometry visual mesh filename=/home/tuan/projects/cibo/3rd_party/GR00T-WholeBodyControl/g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
- link right_shoulder_yaw_link: geometry collision cylinder length=0.13 radius=0.035; visual mesh filename=/home/tuan/projects/cibo/3rd_party/GR00T-WholeBodyControl/g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
- link right_wrist_pitch_link: geometry visual mesh filename=/home/tuan/projects/cibo/3rd_party/GR00T-WholeBodyControl/g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
- link right_wrist_roll_link: geometry visual mesh filename=/home/tuan/projects/cibo/3rd_party/GR00T-WholeBodyControl/g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
- link right_wrist_yaw_link: geometry collision mesh filename=/home/tuan/projects/cibo/3rd_party/GR00T-WholeBodyControl/g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; visual mesh filename=/home/tuan/projects/cibo/3rd_party/GR00T-WholeBodyControl/g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
- link torso_link: geometry collision cylinder length=0.01 radius=0.068; collision cylinder length=0.04 radius=0.065
- link waist_roll_link: geometry visual mesh filename=/home/tuan/projects/cibo/3rd_party/GR00T-WholeBodyControl/g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
- link waist_yaw_link: geometry visual mesh filename=/home/tuan/projects/cibo/3rd_party/GR00T-WholeBodyControl/g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
